Commit message: kautham

File: kautham/square_fixture.urdf (robot description, URDF)
Before this commit: robot square_fixture, 1 links, 0 joints
Links:
- link base_link: geometry collision box size=0.058 0.058 0.075; visual box size=0.058 0.058 0.075

Commit message: fixture taller

File: kautham/square_fixture.urdf (robot description, URDF)
Before this commit: robot square_fixture, 1 links, 0 joints
Links:
- link base_link: geometry collision box size=0.058 0.058 0.125; visual box size=0.058 0.058 0.125

Commit message: movimiento fluido

File: kautham/square_fixture.urdf (robot description, URDF)
Before this commit: robot square_fixture, 1 links, 0 joints
Links:
- link base_link: geometry collision box size=0.058 0.058 0.155; visual box size=0.058 0.058 0.155

Commit message: aa

File: kautham/square_fixture.urdf (robot description, URDF)
Before this commit: robot square_fixture, 1 links, 0 joints
Links:
- link base_link: geometry collision box size=0.058 0.078 0.165; visual box size=0.058 0.078 0.165

Commit message: aaa

File: kautham/square_fixture.urdf (robot description, URDF)
Before this commit: robot square_fixture, 1 links, 0 joints
Links:
- link base_link: geometry collision box size=0.158 0.158 0.105; visual box size=0.158 0.158 0.105

Commit message: aaa

File: kautham/square_fixture.urdf (robot description, URDF)
Before this commit: robot square_fixture, 1 links, 0 joints
Links:
- link base_link: geometry collision box size=0.158 0.158 0.135; visual box size=0.158 0.158 0.135

Commit message: aaa

File: kautham/square_fixture.urdf (robot description, URDF)
Before this commit: robot square_fixture, 1 links, 0 joints
Links:
- link base_link: geometry collision box size=0.158 0.158 0.175; visual box size=0.158 0.158 0.175
